Commit message: modified launch and split_joint_states

File: ur_pers_lib_pkg/xacro/dual_ur_robotiq.xacro (robot description, xacro)
@@ -2,6 +2,6 @@
 <robot xmlns:xacro="http://www.ros.org/wiki/xacro" name="dual">
     <xacro:arg name="simulation" default="true"/>
-    <xacro:arg name="robot1_name" default="1"/>
-    <xacro:arg name="robot2_name" default="2"/>
+    <xacro:arg name="robot1_name" default="right"/>
+    <xacro:arg name="robot2_name" default="left"/>
     <xacro:arg name="robot1_active" default="true"/>
     <xacro:arg name="robot2_active" default="true"/>
@@ -23,4 +23,7 @@
     <xacro:arg name="finger1" default="tactile2x6.STL"/>
     <xacro:arg name="finger2" default="tactile2x6.STL"/>
+    <xacro:arg name="robot1_hw_interface" default="hardware_interface/PositionJointInterface"/>
+    <xacro:arg name="robot2_hw_interface" default="hardware_interface/PositionJointInterface"/>
+    <xacro:arg name="gripper_hw_interface" default="hardware_interface/PositionJointInterface"/>
     <!-- Include URDFs -->
     <xacro:include filename="$(find ur_description)/urdf/inc/ur5e_macro.xacro"/>
@@ -28,7 +31,7 @@
     <link name="world"/>
   <!-- Spawn the robots -->
-    <xacro:macro name="ur_plus_robotiq" params="prefix parent finger1_path='' finger2_path='' rpy:='0 0 0' xyz:='0 0 0' sim:='True'"> <!-- *origin-->
+    <xacro:macro name="ur_plus_robotiq" params="prefix parent robot_hw_interf gripper_hw_interf finger1_path='' finger2_path='' rpy:='0 0 0' xyz:='0 0 0' sim:='True'"> <!-- *origin-->
         <xacro:ur5e_robot prefix="${prefix}"
-                          transmission_hw_interface="hardware_interface/PositionJointInterface"
+                          transmission_hw_interface="${robot_hw_interf}"
         />
         <xacro:robotiq_hand_e gripper_name="${prefix}"
@@ -38,5 +41,6 @@
                         xyz="0 0 0"
                         rpy="0 -1.57 0"
-                        hardware_interface="hardware_interface/PositionJointInterface"/>
+                        hardware_interface="${gripper_hw_interf}"
+        />
         <joint name="${prefix}world_to_base" type="fixed">
             <parent link="world"/>
@@ -48,4 +52,6 @@
         <xacro:ur_plus_robotiq  prefix="${robot1_prefix}"
                                 parent="world"
+                                robot_hw_interf="$(arg robot1_hw_interface)"
+                                gripper_hw_interf="$(arg gripper_hw_interface)"
                                 finger1_path="$(arg finger1)"
                                 finger2_path="$(arg finger2)"
@@ -57,4 +63,6 @@
         <xacro:ur_plus_robotiq  prefix="${robot2_prefix}"
                                 parent="world"
+                                robot_hw_interf="$(arg robot2_hw_interface)"
+                                gripper_hw_interf="$(arg gripper_hw_interface)"
                                 finger1_path="$(arg finger1)"
                                 finger2_path="$(arg finger2)"

Commit message: added diasable gravity

File: ur_pers_lib_pkg/xacro/dual_ur_robotiq.xacro (robot description, xacro)
@@ -48,4 +48,24 @@
             <origin xyz="${xyz}" rpy="${rpy}"/>
         </joint>
+        <!-- disable gravity for links-->
+        <gazebo reference="${prefix}shoulder_link">
+            <gravity>false</gravity>
+        </gazebo>
+        <gazebo reference="${prefix}upper_arm_link">
+            <gravity>false</gravity>
+        </gazebo>
+        <gazebo reference="${prefix}forearm_link">
+            <gravity>false</gravity>
+        </gazebo>
+        <gazebo reference="${prefix}wrist_1_link">
+            <gravity>false</gravity>
+        </gazebo>
+        <gazebo reference="${prefix}wrist_2_link">
+            <gravity>false</gravity>
+        </gazebo>
+        <gazebo reference="${prefix}wrist_3_link">
+            <gravity>false</gravity>
+        </gazebo>
+    </xacro:macro>
     </xacro:macro>
     <xacro:if value="$(arg robot1_active)">

Commit message: fixed bug on xacro

File: ur_pers_lib_pkg/xacro/dual_ur_robotiq.xacro (robot description, xacro)
@@ -68,5 +68,4 @@
         </gazebo>
     </xacro:macro>
-    </xacro:macro>
     <xacro:if value="$(arg robot1_active)">
         <xacro:ur_plus_robotiq  prefix="${robot1_prefix}"
